File: 30-sec-timer.sch (KiCad schematic (older format))
At the start: 21 parts, among them P1 6.3V AC IN, P2 CL12345, P3 Right, P4 Left, Q1 BC557, Q2 BC547, U1 LM7805CT, U2 LM555N

Commit message: relay driveing fix, resistor values fix, added two resistors for led, led brightness fix
Parts:
- added R6: 220, Resistors_THT:R_Axial_DIN0207_L6.3mm_D2.5mm_P7.62mm_Horizontal, symbol R
- added R7: 10K, Resistors_THT:R_Axial_DIN0207_L6.3mm_D2.5mm_P7.62mm_Horizontal, symbol R
- R2: value 10K -> 7K5
- R5: value 1K -> 2K2
Connections:
- net Earth: now also D3.2 (K), Q2.3 (E), R7.2; no longer D4.2 (A), R4.2, RL1.12
- net VCC: now also D4.1 (K), RL1.1; no longer Q2.1 (C)
- net at R2.2, R5.2, U2.3 (Q): now also R6.1; no longer D3.1 (A1)
- net at R4.1: now also Q1.1 (C); no longer D3.2 (K)
- net at D3.3 (A2): now also R4.2; no longer Q1.1 (C)
- net at Q2.2 (B), R5.1: now also R7.1
- new net: D3.1 (A1), R6.2
- new net: D4.2 (A), Q2.1 (C), RL1.12
Other:
- moved on the sheet: D3, D4, Q2, R4, R5, RL1
